File: ma600a-pcbway-handoff-v0.2/project/kicad/MA600A-RefWinch-Encoder.kicad_pcb (KiCad board)
At the start: 2 copper layers, 28 x 12 mm, 17 parts, among them J1 JST-GH-6, U1 MA600A, U2 MP20056GJ-33

Commit message: Changes after upgrading from kicad 7 to kicad 10
Connections:
- J1 pad 6: (no net) -> unconnected-(J1-RSV-Pad6)
- U1 pad 1: (no net) -> unconnected-(U1-IO1-Pad1)
- U1 pad 11: (no net) -> unconnected-(U1-CK100-Pad11)
- U1 pad 15: (no net) -> unconnected-(U1-IO6-Pad15)
- U1 pad 16: (no net) -> unconnected-(U1-NC-Pad16)
- U1 pad 17: (no net) -> unconnected-(U1-E-PAD-Pad17)
- U1 pad 9: (no net) -> unconnected-(U1-IO5-Pad9)
- U2 pad 4: (no net) -> unconnected-(U2-FB-Pad4)
